Commit message: connect RealSense to last link via camera mount

File: mul_franka_description/robots/panda_arm.urdf.xacro (robot description, xacro)
@@ -6,4 +6,5 @@
   <xacro:arg name="use_fake_hardware" default="false"/>
   <xacro:arg name="fake_sensor_commands" default="false"/>
+  <xacro:arg name="add_realsense" default="false"/>
   <xacro:include filename="$(find franka_description)/robots/panda_arm.xacro"/>
   <xacro:panda_arm arm_id="$(arg arm_id)" safety_distance="0.03"/>
@@ -27,3 +28,14 @@
     </xacro:if>
   </xacro:if>
+  <!-- RealSense camera -->
+  <xacro:if value="$(arg add_realsense)">
+    <!-- RealSense camera mount -->
+    <xacro:include filename="$(find mul_franka_description)/robots/panda_realsense_d435_camera_mount.xacro"/>
+    <xacro:panda_realsense_d435_camera_mount arm_id="$(arg arm_id)" connected_to="$(arg arm_id)_link8" xyz="0 0 0.0075" rpy="0 0 ${pi*3/4}"/>
+    <!-- RealSense camera -->
+    <xacro:include filename="$(find realsense2_description)/urdf/_d435.urdf.xacro" />
+    <xacro:sensor_d435 name="$(arg arm_id)_realsense" parent="$(arg arm_id)_realsense_mount_tip" use_nominal_extrinsics="false" add_plug="true" use_mesh="true">
+        <origin xyz="0.010025 0 -0.0115" />
+    </xacro:sensor_d435>
+  </xacro:if>
 </robot>

Commit message: connect RealSense to last link via camera mount

File: mul_franka_description/robots/panda_arm.urdf.xacro (robot description, xacro)
@@ -6,4 +6,5 @@
   <xacro:arg name="use_fake_hardware" default="false"/>
   <xacro:arg name="fake_sensor_commands" default="false"/>
+  <xacro:arg name="add_realsense" default="false"/>
   <xacro:include filename="$(find franka_description)/robots/panda_arm.xacro"/>
   <xacro:panda_arm arm_id="$(arg arm_id)" safety_distance="0.03"/>
@@ -27,3 +28,15 @@
     </xacro:if>
   </xacro:if>
+  <!-- RealSense camera -->
+  <xacro:if value="$(arg add_realsense)">
+    <!-- RealSense camera mount -->
+    <xacro:include filename="$(find mul_franka_description)/robots/panda_realsense_d435_camera_mount.xacro"/>
+    <xacro:panda_realsense_d435_camera_mount arm_id="$(arg arm_id)" connected_to="$(arg arm_id)_link8" xyz="0 0 0.0075" rpy="0 0 ${pi*3/4}"/>
+    <!-- RealSense camera -->
+    <!-- NOTE: The macro argument "name" has to match the parameter "camera_name" of the RealSense node. -->
+    <xacro:include filename="$(find realsense2_description)/urdf/_d435.urdf.xacro" />
+    <xacro:sensor_d435 name="camera" parent="$(arg arm_id)_realsense_mount_tip" use_nominal_extrinsics="false" add_plug="false" use_mesh="true">
+        <origin xyz="0.010025 0 -0.0115" />
+    </xacro:sensor_d435>
+  </xacro:if>
 </robot>
